File: PCB/RPiPicoStand/V02/RaPiPiMiStV02.kicad_pcb (KiCad board)
At the start: 4 copper layers, 55.5 x 73 mm, 20 parts, among them U1-PICO W Pico

Commit message: silkboard updates
Parts:
- added G***: LOGO, LOGO, B.Cu at (195.0, 102.8)
- added G***: LOGO, LOGO, B.Cu at (183.6, 76.0)
- added G***: LOGO, LOGO, B.Cu at (152.0, 85.2)
- added G***: LOGO, LOGO, B.Cu at (171.5, 114.5)
- added G***: LOGO, LOGO, B.Cu at (183.5, 96.0)
- added G***: LOGO, LOGO, B.Cu at (162.8, 57.8)
- added G***: LOGO, LOGO, B.Cu at (160.2, 107.0)
- moved G*** 2.17 mm to (180.8, 119.2)
- moved G*** 0.56 mm to (179.3, 120.0)

Commit message: add teardrops, fix planes
Routing:
- net Net-(5VBUCK2-OUT+): track 48.7 -> 180.9 mm
- added copper zone on B.Cu, net GND
- added copper zone on F.Cu, net GND
- removed copper zone on In1.Cu, net GND
- removed copper zone on F.Cu, net Net-(5VBUCK2-OUT+)

Commit message: fix name of the pcb
Other:
- board text added: "Rappic Micsta v2.0"
- board text removed: "RaPiPiMiSt v2.0"
